File: pcb/untitled.brd (EAGLE design)
At the start: 160 x 100 mm, 6 parts

Commit message: pcb
Parts:
- added C1, C2, C3, C4, C5, C6, C7: 100n, pcb_control_esp:C025-025X050
- added G1: CR2032H, pcb_control_esp:CR2032H
- added IC1: AT24CP, pcb_control_esp:DIL08
- added IC2: 74HC14D, 74xx-eu:SO14
- added IC3: 74HC595D, 74xx-eu:SO16
- added IC4: REG1117, pcb_control_esp:SOT223
- added LED1: (no value), pcb_control_esp:LED3MM
- added Q1: BC548, pcb_control_esp:TO92-EBC
- added R4, R5: (no value), resistor:0207/7
- added SG2: F/EE17P, buzzer:F/EE17P
- added U$2: DS3231SN, pcb_control_esp:SO16W
- added U1: ESP-WROOM-32, ESP32:ESP-WROOM-32
- added X1: SMA-J502-ND, pcb_control_esp:J502-ND
- R1, R2: value 10k -> 4k7; device rcl:0207/10 -> resistor:0207/7
- R3: value 10k -> 4k; device rcl:0207/10 -> resistor:0207/7
- U$1: value ESP32DEVKITV1 -> DFPLAYER-MINI-MODULE; device ESP32-DEVKITV1:ESP32-DEVKITV1 -> pcb_control_esp:DFPLAYER-MINI-MODULE
- moved SV1 87.3 mm to (81.9, 45.1)
- moved SV2 62.1 mm to (95.9, 27.3), turned to 90 degrees
- moved R3 52.3 mm to (75.6, 31.1), turned to 90 degrees
- moved R2 49.7 mm to (72.4, 31.1), turned to 90 degrees
- moved U$1 48.3 mm to (12.7, 37.5), turned to 0 degrees
- moved R1 47.6 mm to (69.2, 31.8), turned to 90 degrees
Connections:
- new net 3V3: U1.2
- new net BUZER: R5.1
- new net CLK: IC2.11
- new net DFRX: U$1.2
- new net DFTX: U$1.3
- new net N$11: IC2.12, IC3.14
- new net N$12: IC2.10, IC3.11, SV1.1
- new net N$13: IC2.8, IC3.12, SV1.3
- new net N$14: IC3.15, SV1.15
- new net N$15: IC3.1, SV1.13
- new net N$16: IC3.2, SV1.11
- new net N$17: IC3.3, SV1.9
- new net N$18: IC2.2, SV1.8
- new net N$19: IC3.9, SV1.10
- new net N$4: Q1.C, SG2.1
- new net N$5: C4.1, G1.+, U$2.14
- new net N$6: Q1.B, R5.2
- new net N$7: LED1.A, R4.1
- new net PINOE: IC2.1
- new net R_DATA: IC2.13
- new net SCL: IC1.6, R3.1, U$2.16
- new net SDA: IC1.5, R2.1, U$2.15
- new net SQW: R1.1, U$2.3
- new net STB: IC2.9
- new net VCC: IC2.14, IC3.16, U$1.1
- net +3V3: now also C3.1, C5.2, C6.1, C7.1, IC1.8, IC4.2, R4.2, U$2.2; no longer U$1.1
- net +5V: now also C1.1, C2.1, IC3.10, IC4.3, SG2.2; no longer U$1.30
- net GND: now also C1.2, C2.2, C3.2, C4.2, C5.1, C6.2, C7.2, G1.-, IC1.1, IC1.2, IC1.3, IC1.4, IC2.7, IC3.13, IC3.8, IC4.1, LED1.K, Q1.E, SV1.12, SV1.14, SV1.16, SV1.2, SV1.4, U$1.10, U$1.7, U$2.10, U$2.11, U$2.12, U$2.13, U$2.4, U$2.5, U$2.6, U$2.7, U$2.8, U$2.9, U1.1, U1.15, U1.38, U1.GND
- net N$1: no longer R1.1, SV2.8, U$1.23
- net N$2: no longer R2.1, SV2.6, U$1.24
- net N$3: no longer R3.1, SV2.4, U$1.24
Other:
- board size 160 x 100 mm -> 100 x 50 mm

Commit message: relayout
Parts:
- added H1, H2, H3, H4: MOUNT-PAD-ROUND3.0, holes:3,0-PAD
- added SV3: (no value), con-lstb:MA03-1
- added SV4: (no value), con-lsta:FE08-2
- moved SV2 70.2 mm to (27.9, 45.1), turned to 180 degrees
- moved SV1 68.5 mm to (15.2, 29.2), turned to 270 degrees
- moved IC3 61.1 mm to (23.5, 29.8), flipped to the bottom, turned to 90 degrees
- moved IC2 59.7 mm to (24.8, 31.8), turned to 90 degrees
- moved C4 54.6 mm to (82.5, 25.4)
- moved IC4 35.2 mm to (31.8, 8.89), turned to 180 degrees
- moved C3 34.2 mm to (38.7, 47.6), turned to 180 degrees
- moved U$1 32.1 mm to (32.4, 12.1), turned to 90 degrees
- moved R5 29.6 mm to (63.5, 21.0), turned to 270 degrees
- moved LED1 24.7 mm to (18.4, 14.6), turned to 90 degrees
- moved R1 20.2 mm to (87.6, 23.5)
- moved C2 20.1 mm to (30.5, 15.9)
- moved R4 19.9 mm to (38.1, 12.7)
- moved C6 19.7 mm to (68.6, 25.4)
- moved R2 19.3 mm to (90.2, 23.5)
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Connections:
- removed net 3V3: U1.2
- new net ENA: U1.4
- new net ENB: U1.5
- new net MNU: U1.6
- new net RELAY: SV3.1
- net +3V3: now also U1.2
- net +5V: now also SV3.2
- net CLK: now also U1.13
- net GND: now also SV3.3
- net R_DATA: now also U1.16
- net SCL: now also U1.36
- net SDA: now also U1.33
- net SQW: now also U1.7
Routing:
- net GND: track 0.00 -> 307.7 mm

Commit message: layout pcb
Parts:
- added C8: 100n, pcb_control_esp:C025-025X050
- added C9: 100u/10, rcl:E2,5-5
- added D1: 1n4002, diode:DO35-10
- added DOWNLOADER: (no value), con-lstb:MA06-1
- added X2: (no value), con-ptr500:AK500/2-H
- C3: value 100n -> 100u/16; device pcb_control_esp:C025-025X050 -> rcl:E2,5-6
- R4, R5: value (none) -> 220
- moved C3 39.3 mm to (18.4, 14.0), turned to 90 degrees
- moved C6 38.8 mm to (35.6, 45.7), turned to 270 degrees
- moved LED1 24.1 mm to (40.0, 25.4), turned to 0 degrees
- moved C2 23.1 mm to (24.1, 38.1), turned to 180 degrees
- moved C4 14.0 mm to (68.6, 24.8), turned to 180 degrees
- moved SG2 13.7 mm to (52.7, 20.3), turned to 180 degrees
- moved Q1 12.7 mm to (57.8, 7.62), turned to 90 degrees
- moved R5 9.71 mm to (61.6, 11.4)
- moved U1 3.81 mm to (48.3, 41.9)
- moved C5 2.29 mm to (33.7, 17.1)
- moved C7 1.42 mm to (97.2, 21.6), turned to 90 degrees
- moved SV2 1.42 mm to (26.7, 45.7)
- moved R1 1.27 mm to (88.9, 23.5)
- moved R3 1.27 mm to (94.0, 23.5)
- moved IC1 1.27 mm to (93.3, 13.3)
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Connections:
- new net N$20: IC2.4, SV2.4
- new net N$8: U$1.6, X2.2
- new net N$9: U$1.8, X2.1
- new net STB_SEG: IC2.3
- net +3V3: now also C8.1, C9.+; no longer C3.1
- net +5V: now also D1.A, DOWNLOADER.2, X1.3, X1.4; no longer IC4.3
- net GND: now also C3.-, C8.2, C9.-, DOWNLOADER.1, SV4.10, SV4.12, SV4.14, SV4.16, SV4.4, SV4.6, SV4.8, X1.2, X1.5; no longer C3.2
- net N$11: now also SV2.6
- net N$12: now also SV2.8, SV4.9
- net N$13: now also SV4.7
- net N$14: now also SV4.15
- net N$15: now also SV4.13
- net N$18: now also SV4.2
- net N$19: now also SV4.5
- net VCC: now also C3.+, D1.C, IC4.3
Routing:
- net GND: track 307.7 -> 459.8 mm
- net +3V3: track 0.00 -> 48.3 mm
- net SDA: track 0.00 -> 31.7 mm
- net VCC: track 0.00 -> 30.4 mm, vias 0 -> 1
- net +5V: track 0.00 -> 27.2 mm
- net SCL: track 0.00 -> 26.2 mm
- net N$14: track 0.00 -> 25.0 mm
- net N$18: track 0.00 -> 21.7 mm
- net SQW: track 0.00 -> 21.5 mm, vias 0 -> 1
- net N$12: track 0.00 -> 21.4 mm
- net N$13: track 0.00 -> 18.9 mm
- net N$15: track 0.00 -> 16.2 mm
- net N$5: track 0.00 -> 15.6 mm
- net N$19: track 0.00 -> 11.6 mm
- net N$16: track 0.00 -> 4.44 mm
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