File: pcb/untitled.sch (EAGLE design)
At the start: 6 parts

Commit message: pcb
Parts:
- added C1, C2, C3, C4, C5, C6, C7: 100n, pcb_control_esp:C-EU025-025X050
- added G1: CR2032H, pcb_control_esp:CR2032H
- added IC1: AT24CP, pcb_control_esp:AT24CP
- added IC2: 74HC14D, 74xx-eu:74HC14D
- added IC3: 74HC595D, 74xx-eu:74HC595D
- added IC4: REG1117, pcb_control_esp:REG1117
- added LED1: (no value), pcb_control_esp:LED3MM
- added Q1: BC548, pcb_control_esp:BC548
- added R4, R5: (no value), resistor:R-EU_0207/7
- added SG2: F/EE17P, buzzer:F/EE17P
- added U$2: DS3231SN, pcb_control_esp:DS3231SN
- added U1: ESP-WROOM-32, ESP32:ESP-WROOM-32
- added X1: SMA-J502-ND, pcb_control_esp:SMA-J502-ND
- R1, R2: value 10k -> 4k7; device rcl:R-EU_0207/10 -> resistor:R-EU_0207/7
- R3: value 10k -> 4k; device rcl:R-EU_0207/10 -> resistor:R-EU_0207/7
- U$1: value ESP32DEVKITV1 -> DFPLAYER-MINI-MODULE; device ESP32-DEVKITV1:ESP32DEVKITV1 -> pcb_control_esp:DFPLAYER-MINI-MODULE
Connections:
- new net BUZER: R5.1
- new net CLK: IC2B.I
- new net DFRX: U$1.RX
- new net DFTX: U$1.TX
- new net N$11: IC2A.O, IC3A.SER
- new net N$12: IC2B.O, IC3A.SCK, SV1.1
- new net N$13: IC2C.O, IC3A.RCK, SV1.3
- new net N$14: IC3A.QA, SV1.15
- new net N$15: IC3A.QB, SV1.13
- new net N$16: IC3A.QC, SV1.11
- new net N$17: IC3A.QD, SV1.9
- new net N$18: IC2D.O, SV1.8
- new net N$19: IC3A.QH*, SV1.10
- new net N$4: Q1.C, SG2.1
- new net N$5: C4.1, G1.+, U$2.VBAT
- new net N$6: Q1.B, R5.2
- new net N$7: LED1.A, R4.1
- new net PINOE: IC2D.I
- new net R_DATA: IC2A.I
- new net SCL: IC1.SCL, R3.1, U$2.SCL
- new net SDA: IC1.SDA, R2.1, U$2.SDA
- new net SQW: R1.1, U$2.!INT/SQW
- new net STB: IC2C.I
- new net VCC: U$1.VCC
- net +3V3: now also C3.1, C5.2, C6.1, C7.1, IC1.VCC, IC4.VOUT, R4.2, U$2.VCC; no longer U$1.3V3
- net +5V: now also C1.1, C2.1, IC3A.SCL, IC4.VIN, SG2.2; no longer U$1.VIN
- net GND: now also C1.2, C2.2, C3.2, C4.2, C5.1, C6.2, C7.2, G1.-, IC1.A0, IC1.A1, IC1.A2, IC1.GND, IC3A.G, IC4.GND, LED1.C, Q1.E, SV1.12, SV1.14, SV1.16, SV1.2, SV1.4, U$1.GND.1, U$1.GND.2, U$2.!RST, U$2.GND, U$2.NC1, U$2.NC2, U$2.NC3, U$2.NC4, U$2.NC5, U$2.NC6, U$2.NC7, U$2.NC8
- net N$1: no longer R1.1, SV2.8, U$1.IO25
- net N$2: no longer R2.1, SV2.6, U$1.IO26
- net N$3: no longer R3.1, SV2.4, U$1.IO27
Other:
- moved on the sheet: R1, R2, R3, SV1, SV2

Commit message: relayout
Parts:
- added H1, H2, H3, H4: MOUNT-PAD-ROUND3.0, holes:MOUNT-PAD-ROUND3.0
- added SV3: (no value), con-lstb:MA03-1
- added SV4: (no value), con-lsta:FE08-2
Connections:
- new net ENA: U1.SENSOR_VP
- new net ENB: U1.SENSOR_VN
- new net MNU: U1.IO34
- new net RELAY: SV3.1
- net +3V3: now also U1.3V3
- net +5V: now also SV3.2
- net CLK: now also U1.IO14
- net GND: now also SV3.3, U1.GND@1, U1.GND@3
- net R_DATA: now also U1.IO13
- net SCL: now also U1.IO22
- net SDA: now also U1.IO21
- net SQW: now also U1.IO35
Changed lines of the file:
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@@
 <part name="C6" library="pcb_control_esp" deviceset="C-EU" device="025-025X050" value="100n"/>
 <part name="C7" library="pcb_control_esp" deviceset="C-EU" device="025-025X050" value="100n"/>
+<part name="GND20" library="supply1" deviceset="GND" device=""/>
+<part name="+3V7" library="pcb_control_esp" deviceset="+3V3" device=""/>
+<part name="+3V8" library="pcb_control_esp" deviceset="+3V3" device=""/>
+<part name="GND21" library="supply1" deviceset="GND" device=""/>
+<part name="SV3" library="con-lstb" deviceset="MA03-1" device=""/>
+<part name="GND22" library="supply1" deviceset="GND" device=""/>
+<part name="P+7" library="supply1" deviceset="+5V" device=""/>
+<part name="H1" library="holes" deviceset="MOUNT-PAD-ROUND" device="3.0"/>
+<part name="H2" library="holes" deviceset="MOUNT-PAD-ROUND" device="3.0"/>
+<part name="H3" library="holes" deviceset="MOUNT-PAD-ROUND" device="3.0"/>
+<part name="H4" library="holes" deviceset="MOUNT-PAD-ROUND" device="3.0"/>
+<part name="SV4" library="con-lsta" deviceset="FE08-2" device=""/>
 </parts>
 <sheets>
@@
 <instance part="C6" gate="G$1" x="304.8" y="-251.46"/>
 <instance part="C7" gate="G$1" x="294.64" y="-251.46"/>
+<instance part="GND20" gate="1" x="40.64" y="-139.7" rot="R270"/>
+<instance part="+3V7" gate="G$1" x="48.26" y="-129.54"/>
+<instance part="+3V8" gate="G$1" x="93.98" y="-132.08"/>
+<instance part="GND21" gate="1" x="99.06" y="-137.16" rot="R90"/>
+<instance part="SV3" gate="G$1" x="-116.84" y="-172.72" rot="MR180"/>
+<instance part="GND22" gate="1" x="-104.14" y="-185.42"/>
+<instance part="P+7" gate="1" x="-104.14" y="-162.56"/>
+<instance part="H1" gate="G$1" x="266.7" y="-86.36"/>
+<instance part="H2" gate="G$1" x="269.24" y="-93.98"/>
+<instance part="H3" gate="G$1" x="269.24" y="-101.6"/>
+<instance part="H4" gate="G$1" x="269.24" y="-109.22"/>
+<instance part="SV4" gate="G$1" x="-48.26" y="-71.12"/>
 </instances>
 <busses>
@@
 <junction x="299.72" y="-246.38"/>
 <pinref part="+3V2" gate="G$1" pin="+3V3"/>
+</segment>
+<segment>
+<pinref part="U1" gate="G$1" pin="3V3"/>
+<pinref part="+3V7" gate="G$1" pin="+3V3"/>
+<wire x1="53.34" y1="-144.78" x2="48.26" y2="-144.78" width="0.1524" layer="91"/>
+<wire x1="48.26" y1="-144.78" x2="48.26" y2="-132.08" width="0.1524" layer="91"/>
 </segment>
 </net>
@@
 <pinref part="GND19" gate="1" pin="GND"/>
 </segment>
+<segment>
+<pinref part="U1" gate="G$1" pin="GND@1"/>
+<wire x1="53.34" y1="-142.24" x2="50.8" y2="-142.24" width="0.1524" layer="91"/>
+<wire x1="50.8" y1="-142.24" x2="50.8" y2="-139.7" width="0.1524" layer="91"/>
+<pinref part="GND20" gate="1" pin="GND"/>
+<wire x1="50.8" y1="-139.7" x2="43.18" y2="-139.7" width="0.1524" layer="91"/>
+</segment>
+<segment>
+<pinref part="U1" gate="G$1" pin="GND@3"/>
+<wire x1="88.9" y1="-142.24" x2="91.44" y2="-142.24" width="0.1524" layer="91"/>
+<wire x1="91.44" y1="-142.24" x2="91.44" y2="-137.16" width="0.1524" layer="91"/>
+<pinref part="GND21" gate="1" pin="GND"/>
+<wire x1="91.44" y1="-137.16" x2="96.52" y2="-137.16" width="0.1524" layer="91"/>
+</segment>
+<segment>
+<pinref part="GND22" gate="1" pin="GND"/>
+<wire x1="-104.14" y1="-175.26" x2="-104.14" y2="-182.88" width="0.1524" layer="91"/>
+<pinref part="SV3" gate="G$1" pin="3"/>
+<wire x1="-109.22" y1="-175.26" x2="-104.14" y2="-175.26" width="0.1524" layer="91"/>
+</segment>
 </net>
 <net name="+5V" class="0">
@@
 <junction x="271.78" y="-246.38"/>
 </segment>
+<segment>
+<pinref part="SV3" gate="G$1" pin="2"/>
+<pinref part="P+7" gate="1" pin="+5V"/>
+<wire x1="-109.22" y1="-172.72" x2="-104.14" y2="-172.72" width="0.1524" layer="91"/>
+<wire x1="-104.14" y1="-172.72" x2="-104.14" y2="-165.1" width="0.1524" layer="91"/>
+</segment>
 </net>
 <net name="N$11" class="0">
@@
 <label x="-200.66" y="-60.96" size="1.778" layer="95" rot="R180" xref="yes"/>
 </segment>
+<segment>
+<pinref part="U1" gate="G$1" pin="IO13"/>
+<wire x1="53.34" y1="-182.88" x2="35.56" y2="-182.88" width="0.1524" layer="91"/>
+<label x="35.56" y="-182.88" size="1.778" layer="95" rot="R180" xref="yes"/>
+</segment>
 </net>
 <net name="CLK" class="0">
@@
 <wire x1="-185.42" y1="-76.2" x2="-200.66" y2="-76.2" width="0.1524" layer="91"/>
 <label x="-200.66" y="-76.2" size="1.778" layer="95" rot="R180" xref="yes"/>
+</segment>
+<segment>
+<pinref part="U1" gate="G$1" pin="IO14"/>
+<wire x1="53.34" y1="-172.72" x2="33.02" y2="-172.72" width="0.1524" layer="91"/>
+<label x="33.02" y="-172.72" size="1.778" layer="95" rot="R180" xref="yes"/>
 </segment>
 </net>
@@
 <label x="170.18" y="-251.46" size="1.778" layer="95" rot="R180" xref="yes"/>
 </segment>
+<segment>
+<pinref part="U1" gate="G$1" pin="IO35"/>
+<wire x1="53.34" y1="-157.48" x2="40.64" y2="-157.48" width="0.1524" layer="91"/>
+<label x="40.64" y="-157.48" size="1.778" layer="95" rot="R180" xref="yes"/>
+</segment>
 </net>
 <net name="SCL" class="0">
@@
 <label x="228.6" y="-317.5" size="1.778" layer="95" xref="yes"/>
 </segment>
+<segment>
+<pinref part="U1" gate="G$1" pin="IO22"/>
+<wire x1="88.9" y1="-147.32" x2="101.6" y2="-147.32" width="0.1524" layer="91"/>
+<label x="101.6" y="-147.32" size="1.778" layer="95" xref="yes"/>
+</segment>
 </net>
 <net name="SDA" class="0">
@@
 <label x="220.98" y="-320.04" size="1.778" layer="95" xref="yes"/>
 </segment>
+<segment>
+<pinref part="U1" gate="G$1" pin="IO21"/>
+<wire x1="88.9" y1="-154.94" x2="101.6" y2="-154.94" width="0.1524" layer="91"/>
+<label x="101.6" y="-154.94" size="1.778" layer="95" xref="yes"/>
+</segment>
 </net>
 <net name="VCC" class="0">
@@
 </segment>
 </net>
+<net name="RELAY" class="0">
+<segment>
+<pinref part="SV3" gate="G$1" pin="1"/>
+<wire x1="-109.22" y1="-170.18" x2="-91.44" y2="-170.18" width="0.1524" layer="91"/>
+<label x="-91.44" y="-170.18" size="1.778" layer="95" xref="yes"/>
+</segment>
+</net>
+<net name="MNU" class="0">
+<segment>
+<pinref part="U1" gate="G$1" pin="IO34"/>
+<wire x1="53.34" y1="-154.94" x2="30.48" y2="-154.94" width="0.1524" layer="91"/>
+<wire x1="27.94" y1="-154.94" x2="30.48" y2="-154.94" width="0.1524" layer="91"/>
+<label x="27.94" y="-154.94" size="1.778" layer="95" rot="R180" xref="yes"/>
+</segment>
+</net>
+<net name="ENB" class="0">
+<segment>
+<pinref part="U1" gate="G$1" pin="SENSOR_VN"/>
+<wire x1="53.34" y1="-152.4" x2="33.02" y2="-152.4" width="0.1524" layer="91"/>
+<label x="33.02" y="-152.4" size="1.778" layer="95" rot="R180" xref="yes"/>
+</segment>
+</net>
+<net name="ENA" class="0">
+<segment>
+<pinref part="U1" gate="G$1" pin="SENSOR_VP"/>
+<wire x1="53.34" y1="-149.86" x2="38.1" y2="-149.86" width="0.1524" layer="91"/>
+<label x="38.1" y="-149.86" size="1.778" layer="95" rot="R180" xref="yes"/>
+</segment>
+</net>

Commit message: layout pcb
Parts:
- added C8: 100n, pcb_control_esp:C-EU025-025X050
- added C9: 100u/10, rcl:CPOL-EUE2.5-5
- added D1: 1n4002, diode:1N4148DO35-10
- added DOWNLOADER: (no value), con-lstb:MA06-1
- added X2: (no value), con-ptr500:AK500/2-H
- C3: value 100n -> 100u/16; device pcb_control_esp:C-EU025-025X050 -> rcl:CPOL-EUE2.5-6
- R4, R5: value (none) -> 220
Connections:
- new net N$20: IC2E.O, SV2.4
- new net N$8: U$1.SPK_1, X2-2.KL
- new net N$9: U$1.SPK_2, X2-1.KL
- new net STB_SEG: IC2E.I
- net +3V3: now also C8.1, C9.+; no longer C3.1
- net +5V: now also D1.A, DOWNLOADER.2, X1.1; no longer IC4.VIN
- net GND: now also C3.-, C8.2, C9.-, DOWNLOADER.1, SV4.10, SV4.12, SV4.14, SV4.16, SV4.4, SV4.6, SV4.8, X1.2; no longer C3.2
- net N$11: now also SV2.6
- net N$12: now also SV2.8, SV4.9
- net N$13: now also SV4.7
- net N$14: now also SV4.15
- net N$15: now also SV4.13
- net N$18: now also SV4.2
- net N$19: now also SV4.5
- net VCC: now also C3.+, D1.C, IC4.VIN
Other:
- moved on the sheet: H1, X1
